Commit message: updated firefly params / max rotors velocity

File: rotors_description/urdf/firefly.xacro (robot description, xacro)
@@ -33,5 +33,6 @@
   <xacro:property name="time_constant_up" value="0.0125" /> <!-- [s] -->
   <xacro:property name="time_constant_down" value="0.025" /> <!-- [s] -->
-  <xacro:property name="max_rot_velocity" value="838" /> <!-- [rad/s] -->
+  <xacro:property name="max_rot_velocity" value="1000" />
+<!-- [rad/s] 838 default -->
   <xacro:property name="sin30" value="0.5" />
   <xacro:property name="cos30" value="0.866025403784" />

Commit message: changed low level controller params

File: rotors_description/urdf/firefly.xacro (robot description, xacro)
@@ -33,6 +33,5 @@
   <xacro:property name="time_constant_up" value="0.0125" /> <!-- [s] -->
   <xacro:property name="time_constant_down" value="0.025" /> <!-- [s] -->
-  <xacro:property name="max_rot_velocity" value="1000" />
-<!-- [rad/s] 838 default -->
+  <xacro:property name="max_rot_velocity" value="838" /> <!-- [rad/s] 838 default -->
   <xacro:property name="sin30" value="0.5" />
   <xacro:property name="cos30" value="0.866025403784" />
